File: EthTInfo.brd (EAGLE design)
At the start: 16.9 x 19 mm, 12 parts, among them J1 1X2-3.5MM-3.5MM, Q1 BSS138

Commit message: Bump to V1.1
Bump to V1.1
Parts:
- removed RGB: SK68051515, _c2h:SK6805-1515
- removed U$3: (no value), _c2h-MacBook Pro de Charles-Henri:LOGO_C2I_015
- added U$2: WS2812-2020SK2020, _c2h:SK6805-2020
- moved R1 2.40 mm to (13.8, 18.3), turned to 180 degrees
- moved Q1 1.55 mm to (12.8, 20.2), turned to 90 degrees
- moved R4 0.76 mm to (9.14, 21.6)
- moved TRM1 0.25 mm to (14.1, 8.13)
- moved C1 0.16 mm to (10.7, 6.99)
Connections:
- new net N$5: U$2.2
- net 3V3: now also U$2.1; no longer RGB.2
- net GND: now also U$2.3; no longer RGB.4
- net N$6: now also PTH2.10, U$2.4; no longer PTH2.8, RGB.1
Routing:
- net 3V3: track 32.2 -> 30.9 mm
- net N$1: track 4.34 -> 5.29 mm
- net N$6: track 20.3 -> 21.2 mm
Other:
- board text added: "V1.1"
- board text removed: "V1.0"
